File: PCB/STM32_watch_NFC/nfc_rfid.kicad_sch (KiCad schematic)
At the start: 34 parts, among them U3 ST25R3916-AQWT, Y1 27.12Mhz

Commit message: Kicad - Routing 4
Completed version. I just need to add graphics :)
Parts:
- added A1, A2: ~, TestPoint:TestPoint_Pad_D1.5mm, symbol Connector:TestPoint
Connections:
- net A1: now also A1.1
- net A2: now also A2.1
Changed lines of the file:
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@@
   (junction (at 154.94 69.215) (diameter 0) (color 0 0 0 0)
+  )
+  (junction (at 219.71 116.205) (diameter 0) (color 0 0 0 0)
+  )
+  (junction (at 219.71 97.155) (diameter 0) (color 0 0 0 0)
   )
   (junction (at 127.635 111.76) (diameter 0) (color 0 0 0 0)
@@
     )
   )
+  (symbol (lib_id "Connector:TestPoint") (at 219.71 116.205 180) (unit 1)
+    (in_bom yes) (on_board yes) (dnp no)
+    (property "Reference" "A1" (at 222.25 121.285 0)
+      (effects (font (size 1.27 1.27)) (justify left))
+    )
+    (property "Value" "~" (at 229.235 120.65 0)
+      (effects (font (size 1.27 1.27)) (justify left))
+    )
+    (property "Footprint" "TestPoint:TestPoint_Pad_D1.5mm" (at 214.63 116.205 0)
+      (effects (font (size 1.27 1.27)) hide)
+    )
+    (property "Datasheet" "~" (at 214.63 116.205 0)
+      (effects (font (size 1.27 1.27)) hide)
+    )
+    (pin "1")
+    (instances
+      (project "STM32_watch_NFC"
+        (path "/e445874f-c7a3-43dd-b930-6bce1d4fa2ef/282b593a-b5a6-4e14-bd95-457030278cb7"
+          (reference "A1") (unit 1)
+        )
+      )
+    )
+  )
   (symbol (lib_id "Device:C") (at 191.135 88.265 90) (unit 1)
     (in_bom yes) (on_board yes) (dnp no)
@@
         )
       )
+    )
+  )
+  (symbol (lib_id "Connector:TestPoint") (at 219.71 97.155 0) (unit 1)
+    (in_bom yes) (on_board yes) (dnp no)
+    (property "Reference" "A2" (at 216.535 92.075 0)
+      (effects (font (size 1.27 1.27)) (justify left))
+    )
+    (property "Value" "~" (at 210.185 92.71 0)
+      (effects (font (size 1.27 1.27)) (justify left))
+    )
+    (property "Footprint" "TestPoint:TestPoint_Pad_D1.5mm" (at 224.79 97.155 0)
+      (effects (font (size 1.27 1.27)) hide)
+    )
+    (property "Datasheet" "~" (at 224.79 97.155 0)
+      (effects (font (size 1.27 1.27)) hide)
+    )
+    (pin "1")
+    (instances
+      (project "STM32_watch_NFC"
+        (path "/e445874f-c7a3-43dd-b930-6bce1d4fa2ef/282b593a-b5a6-4e14-bd95-457030278cb7"
+          (reference "A2") (unit 1)
+        )
+      )
