File: PCB/STM32_watch_NFC/STM32_watch_NFC.kicad_sch (KiCad schematic)
At the start: 60 parts, among them J1 Conn_01x06_Socket, Q1 2N7000, SW1 SW_DPST_x2, SW2 SW_DPST_x2, SW3 SW_DPST_x2, U1 STM32L031G6Ux, Y2 32.768kHz

Commit message: new branch
Connections:
- net SPI_CS_STM: no longer names the net of U1.10 (PA4)
- net SPI_IRQ_STM: no longer names the net of U1.9 (PA3)
- net SPI_MISO_STM: no longer names the net of U1.12 (PA6)
- net SPI_MOSI_STM: no longer names the net of U1.13 (PA7)
- net SPI_SCL_STM: no longer names the net of U1.11 (PA5)
Other:
- removed sheet NFC_RFID
- added sheet Led_matrix (led_matrix.kicad_sch)

Commit message: NFC is back
Other:
- removed sheet Led_matrix
- added sheet nfc_rfig (nfc_rfid.kicad_sch)
Changed lines of the file:
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@@
 	)
 	(sheet
-		(at 252.73 104.14)
-		(size 12.7 22.86)
+		(at 238.76 102.235)
+		(size 31.75 25.4)
 		(fields_autoplaced yes)
 		(stroke
@@
 			(color 0 0 0 0.0000)
 		)
-		(property "Sheetname" "Led_matrix"
-			(at 252.73 103.4284 0)
+		(property "Sheetname" "nfc_rfig"
+			(at 238.76 101.5234 0)
 			(effects
 				(font
@@
 			)
 		)
-		(property "Sheetfile" "led_matrix.kicad_sch"
-			(at 252.73 127.5846 0)
+		(property "Sheetfile" "nfc_rfid.kicad_sch"
+			(at 238.76 128.2196 0)
 			(effects
 				(font
@@
 			(project "STM32_watch_NFC"
 				(path "/e445874f-c7a3-43dd-b930-6bce1d4fa2ef"
-					(page "2")
+					(page "3")
 				)
 			)
